Commit message: wip

File: rofunc/simulator/assets/urdf/unitreeG1/urdf/g1_29dof.urdf (robot description, URDF)
Before this commit: robot g1_29dof, 40 links, 39 joints
Joints:
- joint left_ankle_pitch_joint: limit lower=-0.87267 upper=0.5236 effort=35 velocity=30 -> lower=-0.87267 upper=0.5236 effort=50 velocity=37
- joint left_ankle_roll_joint: limit lower=-0.2618 upper=0.2618 effort=35 velocity=30 -> lower=-0.2618 upper=0.2618 effort=50 velocity=37
- joint right_ankle_pitch_joint: limit lower=-0.87267 upper=0.5236 effort=35 velocity=30 -> lower=-0.87267 upper=0.5236 effort=50 velocity=37
- joint right_ankle_roll_joint: limit lower=-0.2618 upper=0.2618 effort=35 velocity=30 -> lower=-0.2618 upper=0.2618 effort=50 velocity=37
- joint waist_pitch_joint: limit lower=-0.52 upper=0.52 effort=35 velocity=30 -> lower=-0.52 upper=0.52 effort=50 velocity=37
- joint waist_roll_joint: limit lower=-0.52 upper=0.52 effort=35 velocity=30 -> lower=-0.52 upper=0.52 effort=50 velocity=37
